File: clock.kicad_sch (KiCad schematic)
At the start: 2 parts, among them J4 Conn_01x06_Socket, J5 Conn_01x06_Socket

Commit message: convert to new format
Parts:
- removed J4, J5: Conn_01x06_Socket, Connector_PinSocket_2.54mm:PinSocket_1x06_P2.54mm_Vertical, symbol Connector:Conn_01x06_Socket
- added J4, J5: Conn_01x07_Socket, Connector_PinSocket_2.54mm:PinSocket_1x07_P2.54mm_Vertical, symbol Connector:Conn_01x07_Socket
Connections:
- net +5V: now also J5.7 (Pin_7)
- net Clock1.5: now also J4.7 (Pin_7)
- net Clock12: now also J4.4 (Pin_4)
- net Clock24: now also J4.3 (Pin_3)
- net Clock3: now also J4.6 (Pin_6)
- net Clock6: now also J4.5 (Pin_5)
- net E: now also J5.2 (Pin_2)
- net GND: now also J5.1 (Pin_1)
- net Q: now also J5.5 (Pin_5)
- net ~{E}: now also J5.3 (Pin_3)
- net ~{Q}: now also J5.6 (Pin_6)
- net ~{RESET}: now also J5.4 (Pin_4)
- new net intD0: J4.1 (Pin_1)
- new net intD1: J4.2 (Pin_2)
Other:
- title: (none) -> HD6309 Homebrew SBC
