File: clock.kicad_sch (KiCad schematic)
At the start: 2 parts, among them J4 Conn_01x07_Socket, J5 Conn_01x07_Socket

Commit message: update readme
Connections:
- net intD0 renamed intD00
- net intD1 renamed intD01
Changed lines of the file:
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@@
 (kicad_sch
-	(version 20231120)
+	(version 20250114)
 	(generator "eeschema")
-	(generator_version "8.0")
+	(generator_version "9.0")
 	(paper "A4")
 	(title_block
@@
 		)
 	)
-	(label "intD0"
+	(label "intD00"
 		(at 170.18 59.69 0)
-		(fields_autoplaced yes)
 		(effects
 			(font
@@
 		)
 	)
-	(label "intD1"
+	(label "intD01"
 		(at 170.18 62.23 0)
-		(fields_autoplaced yes)
 		(effects
 			(font
@@
 		)
 	)
-	(hierarchical_label "intD[0..7]"
+	(hierarchical_label "intD0[0..7]"
 		(shape output)
 		(at 166.37 54.61 180)
-		(fields_autoplaced yes)
-		(effects
-			(font
+		(effects
+			(font
