File: control_register_1.kicad_sch (KiCad schematic)
At the start: 8 parts, among them U10 74LS375D, U11 74HC02, U13 74HC21D, U14 74HC21D, U15 74HC21D, U5 74HC08, U7 74HC04D, U9 74LS375D

Commit message: Refine reset circuit
Parts:
- removed U7: 74HC04D, Package_SO:SOIC-14_3.9x8.7mm_P1.27mm, symbol 74xx:74HC04
- added unit 4 of U11
- added U8: 74HC00D, Package_SO:SOIC-14_3.9x8.7mm_P1.27mm, symbol 74xx:74HC00
Connections:
- net R/~{W}: now also U11.11, U11.12
- net Vector: now also U8.1, U8.2
- net at U13.9: now also U11.13
- net at U5.9: now also U8.3
Changed lines of the file:
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@@
+    (stroke (width 0) (type default))
+  )
+  (wire (pts (xy 75.438 40.894) (xy 80.518 40.894))
     (stroke (width 0) (type default))
   )
@@
   )
   (wire (pts (xy 65.532 57.404) (xy 65.532 40.894))
+    (stroke (width 0) (type default))
+  )
+  (wire (pts (xy 112.776 158.496) (xy 112.776 163.576))
     (stroke (width 0) (type default))
   )
@@
     )
   )
+  (symbol (lib_id "74xx:74HC00") (at 120.396 161.036 0) (mirror x) (unit 1)
+    (in_bom yes) (on_board yes) (dnp no) (fields_autoplaced)
+    (property "Reference" "U8" (at 120.396 151.892 0)
+      (effects (font (size 1.27 1.27)))
+    )
+    (property "Value" "74HC00D" (at 120.396 154.432 0)
+      (effects (font (size 1.27 1.27)))
+    )
+    (property "Footprint" "Package_SO:SOIC-14_3.9x8.7mm_P1.27mm" (at 120.396 161.036 0)
+      (effects (font (size 1.27 1.27)) hide)
+    )
+    (property "Datasheet" "http://www.ti.com/lit/gpn/sn74hc00" (at 120.396 161.036 0)
+      (effects (font (size 1.27 1.27)) hide)
+    )
+    (property "DigiKey" "74HC00DCT-ND" (at 120.396 161.036 0)
+      (effects (font (size 1.27 1.27)) hide)
+    )
+    (pin "1")
+    (pin "2")
+    (pin "3")
+    (pin "4")
+    (pin "5")
+    (pin "6")
+    (pin "10")
+    (pin "8")
+    (pin "9")
+    (pin "11")
+    (pin "12")
+    (pin "13")
+    (pin "14")
+    (pin "7")
+    (instances
+      (project "HD6309sbc"
+        (path "/b6976bcd-dc73-4942-aa19-f7adbf9104c7"
+          (reference "U8") (unit 1)
+        )
+        (path "/b6976bcd-dc73-4942-aa19-f7adbf9104c7/c84c6ca6-49e6-40c1-b118-fd043db52510"
+          (reference "U8") (unit 1)
+        )
+      )
+    )
+  )
   (symbol (lib_id "74xx:74LS21") (at 59.182 180.594 0) (unit 2)
     (in_bom yes) (on_board yes) (dnp no)
@@
     )
   )
-  (symbol (lib_id "74xx:74HC04") (at 77.978 48.514 270) (unit 4)
-    (in_bom yes) (on_board yes) (dnp no) (fields_autoplaced)
-    (property "Reference" "U7" (at 82.804 47.2439 90)
-      (effects (font (size 1.27 1.27)) (justify left))
-    )
-    (property "Value" "74HC04D" (at 82.804 49.7839 90)
-      (effects (font (size 1.27 1.27)) (justify left))
-    )
-    (property "Footprint" "Package_SO:SOIC-14_3.9x8.7mm_P1.27mm" (at 77.978 48.514 0)
-      (effects (font (size 1.27 1.27)) hide)
-    )
-    (property "Datasheet" "https://assets.nexperia.com/documents/data-sheet/74HC_HCT04.pdf" (at 77.978 48.514 0)
-      (effects (font (size 1.27 1.27)) hide)
-    )
-    (property "DigiKey" "74HC04DCT-ND" (at 267.462 139.954 90)
-      (effects (font (size 1.27 1.27)) hide)
-    )
-    (pin "1")
-    (pin "2")
-    (pin "3")
-    (pin "4")
-    (pin "5")
-    (pin "6")
-    (pin "8")
-    (pin "9")
-    (pin "10")
-    (pin "11")
-    (pin "12")
-    (pin "13")
-    (pin "14")
-    (pin "7")
-    (instances
-      (project "HD6309sbc"
-        (path "/b6976bcd-dc73-4942-aa19-f7adbf9104c7/c84c6ca6-49e6-40c1-b118-fd043db52510"
-          (reference "U7") (unit 4)
-        )
-      )
-    )
-  )
   (symbol (lib_id "74xx:74LS08") (at 54.102 84.582 0) (unit 4)
     (in_bom yes) (on_board yes) (dnp no) (fields_autoplaced)
@@
     )
   )
-  (symbol (lib_id "74xx:74HC04") (at 120.396 161.036 0) (unit 2)
-    (in_bom yes) (on_board yes) (dnp no) (fields_autoplaced)
-    (property "Reference" "U7" (at 120.396 151.892 0)
-      (effects (font (size 1.27 1.27)))
-    )
-    (property "Value" "74HC04D" (at 120.396 154.432 0)
-      (effects (font (size 1.27 1.27)))
-    )
-    (property "Footprint" "Package_SO:SOIC-14_3.9x8.7mm_P1.27mm" (at 120.396 161.036 0)
-      (effects (font (size 1.27 1.27)) hide)
-    )
-    (property "Datasheet" "https://assets.nexperia.com/documents/data-sheet/74HC_HCT04.pdf" (at 120.396 161.036 0)
-      (effects (font (size 1.27 1.27)) hide)
-    )
-    (property "DigiKey" "74HC04DCT-ND" (at 211.836 -28.448 90)
-      (effects (font (size 1.27 1.27)) hide)
-    )
-    (pin "1")
-    (pin "2")
-    (pin "3")
-    (pin "4")
-    (pin "5")
-    (pin "6")
-    (pin "8")
-    (pin "9")
-    (pin "10")
-    (pin "11")
-    (pin "12")
-    (pin "13")
-    (pin "14")
-    (pin "7")
-    (instances
-      (project "HD6309sbc"
-        (path "/b6976bcd-dc73-4942-aa19-f7adbf9104c7/c84c6ca6-49e6-40c1-b118-fd043db52510"
-          (reference "U7") (unit 2)
-        )
-      )
+  (symbol (lib_id "74xx:74LS02") (at 77.978 48.514 270) (unit 4)
+    (in_bom yes) (on_board yes) (dnp no) (fields_autoplaced)
+    (property "Reference" "U11" (at 82.55 47.879 90)
+      (effects (font (size 1.27 1.27)) (justify left))
+    )
+    (property "Value" "74HC02" (at 82.55 50.419 90)
+      (effects (font (size 1.27 1.27)) (justify left))
+    )
+    (property "Footprint" "Package_SO:SO-14_3.9x8.65mm_P1.27mm" (at 77.978 48.514 0)
+      (effects (font (size 1.27 1.27)) hide)
+    )
+    (property "Datasheet" "http://www.ti.com/lit/gpn/sn74ls02" (at 77.978 48.514 0)
+      (effects (font (size 1.27 1.27)) hide)
+    )
+    (pin "1")
+    (pin "2")
+    (pin "3")
+    (pin "4")
+    (pin "5")
+    (pin "6")
+    (pin "10")
+    (pin "8")
+    (pin "9")
+    (pin "11")
+    (pin "12")
+    (pin "13")
+    (pin "14")
+    (pin "7")
+    (instances
+      (project "HD6309sbc"
+        (path "/b6976bcd-dc73-4942-aa19-f7adbf9104c7"
+          (reference "U11") (unit 4)
+        )
+        (path "/b6976bcd-dc73-4942-aa19-f7adbf9104c7/c84c6ca6-49e6-40c1-b118-fd043db52510"
+          (reference "U11") (unit 4)
+        )
+      )

Commit message: convert to new format
Other:
- note added: "Address range $ff00-$ffef"
- note added: "Address range $fffx"
- note added: "Address range $ffxx"
- note added: "Memory mapping $FF00 : $FFFF reserved for mapped memory $FF00 ... : mapped hardware registers $FFEF $FFF0 ... : interrupt vectors $FFFF"
- note added: "select $ff24 from reserved memory"
