File: diagnostics.kicad_sch (KiCad schematic)
At the start: 28 parts

Commit message: clean up before redesign
Parts:
- added D18, D19, D20, D21, D22, D23, D24, D25: LED_Filled, LED_SMD:LED_1206_3216Metric_Pad1.42x1.75mm_HandSolder, symbol Device:LED_Filled
- added R22, R23, R24, R25, R26, R27, R28, R29: 470R, Resistor_SMD:R_0805_2012Metric_Pad1.20x1.40mm_HandSolder, symbol Device:R_Small
Connections:
- net GND: now also R22.2, R23.2, R24.2, R25.2, R26.2, R27.2, R28.2, R29.2
- net intD0 renamed intD00
- net intD1 renamed intD01
- net intD2 renamed intD02
- net intD3 renamed intD03
- net intD4 renamed intD04
- net intD5 renamed intD05
- net intD6 renamed intD06
- net intD7 renamed intD07
- new net: D18.1 (K), R22.1
- new net: D21.1 (K), R25.1
- new net: D23.1 (K), R27.1
- new net: D22.1 (K), R26.1
- new net: D20.1 (K), R24.1
- new net: D25.1 (K), R29.1
- new net: D24.1 (K), R28.1
- new net: D19.1 (K), R23.1
- new net intD10: D18.2 (A)
- new net intD11: D19.2 (A)
- new net intD12: D20.2 (A)
- new net intD13: D21.2 (A)
- new net intD14: D22.2 (A)
- new net intD15: D23.2 (A)
- new net intD16: D24.2 (A)
- new net intD17: D25.2 (A)
